Commit message: added all joint controllers

File: gazebo/src/robosnake_description/urdf/robosnake.urdf (robot description, URDF)
Before this commit: robot robosnake, 2 links, 1 joints
Links:
- added link segment_00
- added link segment_03
- added link segment_04
- added link segment_05
- added link segment_06
- added link segment_07
- added link segment_08
- added link segment_09
- added link segment_10
- link segment_01: mass 0.4 -> None
- link segment_02: mass 0.4 -> None
Joints:
- added joint joint_0: type revolute, parent segment_00, child segment_01, limit lower=-1.5708 upper=1.5708 effort=100.0 velocity=1
- added joint joint_2: type revolute, parent segment_02, child segment_03, limit lower=-1.5708 upper=1.5708 effort=100.0 velocity=1
- added joint joint_3: type revolute, parent segment_03, child segment_04, limit lower=-1.5708 upper=1.5708 effort=100.0 velocity=1
- added joint joint_4: type revolute, parent segment_04, child segment_05, limit lower=-1.5708 upper=1.5708 effort=100.0 velocity=1
- added joint joint_5: type revolute, parent segment_05, child segment_06, limit lower=-1.5708 upper=1.5708 effort=100.0 velocity=1
- added joint joint_6: type revolute, parent segment_06, child segment_07, limit lower=-1.5708 upper=1.5708 effort=100.0 velocity=1
- added joint joint_7: type revolute, parent segment_07, child segment_08, limit lower=-1.5708 upper=1.5708 effort=100.0 velocity=1
- added joint joint_8: type revolute, parent segment_08, child segment_09, limit lower=-1.5708 upper=1.5708 effort=100.0 velocity=1
- added joint joint_9: type revolute, parent segment_09, child segment_10, limit lower=-1.5708 upper=1.5708 effort=100.0 velocity=1
- joint joint_1: axis 0 0 -1 -> (none); limit lower=-1.5708 upper=1.5708 effort=100.0 velocity=0.2 -> lower=-1.5708 upper=1.5708 effort=100.0 velocity=1; origin xyz=0.007 0 0 rpy= 0 -0 0 -> (none)

Commit message: added real simulation params

File: gazebo/src/robosnake_description/urdf/robosnake.urdf (robot description, URDF)
Before this commit: robot robosnake, 11 links, 10 joints
Joints:
- joint joint_0: limit lower=-1.5708 upper=1.5708 effort=100.0 velocity=1 -> lower=-1.5708 upper=1.5708 effort=17.2886 velocity=1.6936
- joint joint_1: limit lower=-1.5708 upper=1.5708 effort=100.0 velocity=1 -> lower=-1.5708 upper=1.5708 effort=17.2886 velocity=1.6936
- joint joint_2: limit lower=-1.5708 upper=1.5708 effort=100.0 velocity=1 -> lower=-1.5708 upper=1.5708 effort=17.2886 velocity=1.6936
- joint joint_3: limit lower=-1.5708 upper=1.5708 effort=100.0 velocity=1 -> lower=-1.5708 upper=1.5708 effort=17.2886 velocity=1.6936
- joint joint_4: limit lower=-1.5708 upper=1.5708 effort=100.0 velocity=1 -> lower=-1.5708 upper=1.5708 effort=17.2886 velocity=1.6936
- joint joint_5: limit lower=-1.5708 upper=1.5708 effort=100.0 velocity=1 -> lower=-1.5708 upper=1.5708 effort=17.2886 velocity=1.6936
- joint joint_6: limit lower=-1.5708 upper=1.5708 effort=100.0 velocity=1 -> lower=-1.5708 upper=1.5708 effort=17.2886 velocity=1.6936
- joint joint_7: limit lower=-1.5708 upper=1.5708 effort=100.0 velocity=1 -> lower=-1.5708 upper=1.5708 effort=17.2886 velocity=1.6936
- joint joint_8: limit lower=-1.5708 upper=1.5708 effort=100.0 velocity=1 -> lower=-1.5708 upper=1.5708 effort=17.2886 velocity=1.6936
- joint joint_9: limit lower=-1.5708 upper=1.5708 effort=100.0 velocity=1 -> lower=-1.5708 upper=1.5708 effort=17.2886 velocity=1.6936
